Commit message: Gazebo対応だけ動いたrviz未反映バグあり

File: config/sixdofarm.urdf.xacro (robot description, xacro)
@@ -6,4 +6,5 @@
     <!-- Import control_xacro -->
     <xacro:include filename="sixdofarm.ros2_control.xacro" />
+    <!-- ros2_control for simulation -->
     <xacro:sixdofarm_ros2_control name="FakeSystem" initial_positions_file="$(arg initial_positions_file)"/>
 </robot>

File: config/sixdofarm_gazebo.ros2_control.xacro (robot description, xacro)
@@ -1,10 +1,10 @@
 <?xml version="1.0"?>
 <robot xmlns:xacro="http://www.ros.org/wiki/xacro">
-    <xacro:macro name="sixdofarm_ros2_control" params="name initial_positions_file">
+    <xacro:macro name="sixdofarm_gazebo_ros2_control" params="name initial_positions_file">
         <xacro:property name="initial_positions" value="${load_yaml(initial_positions_file)['initial_positions']}"/>
         <ros2_control name="${name}" type="system">
             <hardware>
-                <!-- For simulation with mock hardware -->
-                <plugin>mock_components/GenericSystem</plugin>
+                <!-- For Gazebo simulation -->
+                <plugin>gz_ros2_control/GazeboSimSystem</plugin>
             </hardware>
             <joint name="Link1_2_Link2">
